File: motherboard/V1/MB_V1.kicad_pcb (KiCad board)
At the start: 4 copper layers, 84 x 64 mm, 85 parts, among them IC1 TPS27S100BRRKR, IC2 TPS27S100BRRKR, IC3 TPS27S100BRRKR, IC4 TPS27S100BRRKR, IC5 TPS27S100BRRKR, IC7 STM32L010F4P6TR, J1 640456-6, J2 640456-6, J3 640456-6, J4 640456-6, J5 640454-2, J6 640456-6, Q1 SQS141ELNW-T1_GE3

Commit message: MB_V1 changed
Parts:
- moved R32 8.30 mm to (159.5, 143.4), turned to 90 degrees
- moved F1 3.79 mm to (105.4, 143.2)
- moved IC7 1.33 mm to (158.5, 148.3), turned to -90 degrees
- moved D1 0.40 mm to (105.1, 148.1)
Routing:
- net GND: track 276.2 -> 344.0 mm, vias 59 -> 60
- net Net-(Q1-D_1): track 2.12 -> 16.3 mm
- net /DCDC2_EN: track 47.4 -> 61.3 mm, vias 2 -> 3
- net /DCDC3_EN: track 39.1 -> 52.3 mm, vias 2 -> 3
- net /VCC3: track 33.0 -> 45.5 mm, vias 29 -> 30
- net /S4_SW_EN: track 13.3 -> 24.3 mm, vias 1 -> 2
- net /S3_SW_EN: track 21.4 -> 31.3 mm, vias 1 -> 2
- net /S5_SW_EN: track 5.39 -> 14.7 mm, vias 1 -> 2
- net /S1_SW_IMON: track 38.1 -> 47.0 mm, vias 1 -> 2
- net /S2_SW_EN: track 30.1 -> 38.5 mm, vias 1 -> 2
- net /S1_SW_EN: track 37.4 -> 44.9 mm, vias 1 -> 2
- net /S2_SW_IMON: track 32.8 -> 39.7 mm, vias 1 -> 2
- net /S4_SW_IMON: track 15.0 -> 20.7 mm, vias 1 -> 2
- net /S3_SW_IMON: track 23.8 -> 29.3 mm, vias 1 -> 2
- net /S5_SW_IMON: track 7.71 -> 12.6 mm, vias 1 -> 2
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
Commit message: MB V1 finished
Parts:
- added C13: C0603C104K5RAC3121, SamacSys_Parts:CAPC1608X95N, F.Cu at (162.7, 151.6)
- added G***: LOGO, LOGO, F.Cu at (117.3, 155.0)
- added Q2: IRLML6244TRPBF, SamacSys_Parts:SOT95P237X112-3N, F.Cu at (161.0, 154.6)
- added R48: WSL080500000ZEA9, SamacSys_Parts:RESC2013X84N, F.Cu at (129.5, 123.0)
- added R49: ERJ2RKF1003X, SamacSys_Parts:ERJ2RKD1004X, F.Cu at (158.5, 155.2)
- added R50: ERJ-2RKF1002X, SamacSys_Parts:ERJ2RKD1004X, F.Cu at (162.8, 156.9)
- added R51: ERJ-2RKF1002X, SamacSys_Parts:ERJ2RKD1004X, F.Cu at (153.3, 159.6)
- added R52: ERJ-2RKF1002X, SamacSys_Parts:ERJ2RKD1004X, F.Cu at (154.4, 159.4)
- moved J5 0.40 mm to (99.8, 144.8)
- moved J4 0.07 mm to (120.9, 160.6)
- renumbered H2 to H1, H1 to H2
Connections:
- H1 pad 1: unconnected-(H2-Pad1) -> /VCC3
- H1 pad 100: unconnected-(H2-Pad100) -> GND
- H1 pad 11: unconnected-(H2-Pad11) -> /H3_19
- H1 pad 12: unconnected-(H2-Pad12) -> /H3_18
- H1 pad 13: unconnected-(H2-Pad13) -> /H3_9
- H1 pad 14: unconnected-(H2-Pad14) -> /H3_8
- H1 pad 17: unconnected-(H2-Pad17) -> /PWR_I2C_PULLUP
- H1 pad 2: unconnected-(H2-Pad2) (its old number) -> /VCC3
- H1 pad 25: unconnected-(H2-Pad25) -> GND
- H1 pad 26: unconnected-(H2-Pad26) -> /VCC2_OUT
- H1 pad 30: unconnected-(H2-Pad30) -> /H3_14
- H1 pad 31: unconnected-(H2-Pad31) -> /H3_13
- H1 pad 32: unconnected-(H2-Pad32) -> /H3_12
- H1 pad 36: unconnected-(H2-Pad36) -> /H4_19
- H1 pad 37: unconnected-(H2-Pad37) -> /H4_18
- H1 pad 38: unconnected-(H2-Pad38) -> /H4_7
- H1 pad 39: unconnected-(H2-Pad39) -> /H4_6
- H1 pad 4: unconnected-(H2-Pad4) -> /H4_17
- H1 pad 40: unconnected-(H2-Pad40) -> /H3_15
- H1 pad 5: unconnected-(H2-Pad5) -> /H4_16
- H1 pad 50: unconnected-(H2-Pad50) -> GND
- H1 pad 51: unconnected-(H2-Pad51) -> GND
- H1 pad 54: unconnected-(H2-Pad54) -> /H2_9
- H1 pad 55: unconnected-(H2-Pad55) -> /H2_8
- H1 pad 6: unconnected-(H2-Pad6) -> /H4_15
- H1 pad 61: unconnected-(H2-Pad61) -> /H3_17
- H1 pad 62: unconnected-(H2-Pad62) -> /H3_16
- H1 pad 64: unconnected-(H2-Pad64) -> /PWR_MCU_I2C_SDA
- H1 pad 65: unconnected-(H2-Pad65) -> /PWR_MCU_I2C_SCL
- H1 pad 66: unconnected-(H2-Pad66) -> /H5_17
- H1 pad 67: unconnected-(H2-Pad67) -> /H5_16
- H1 pad 68: unconnected-(H2-Pad68) -> /H5_15
- H1 pad 7: unconnected-(H2-Pad7) -> /PWR_MCU_BOOTLOADER
- H1 pad 75: unconnected-(H2-Pad75) -> GND
- H1 pad 76: unconnected-(H2-Pad76) -> GND
- H1 pad 78: unconnected-(H2-Pad78) -> /H2_16
- H1 pad 79: unconnected-(H2-Pad79) -> /H2_15
- H1 pad 80: unconnected-(H2-Pad80) -> /H3_7
- H1 pad 81: unconnected-(H2-Pad81) -> /H3_6
- H1 pad 82: unconnected-(H2-Pad82) -> /H2_14
- H1 pad 83: unconnected-(H2-Pad83) -> /H2_13
- H1 pad 84: unconnected-(H2-Pad84) -> /H2_12
- H1 pad 85: unconnected-(H2-Pad85) -> /H2_19
- H1 pad 86: unconnected-(H2-Pad86) -> /H2_7
- H1 pad 87: unconnected-(H2-Pad87) -> /H2_6
- H1 pad 88: unconnected-(H2-Pad88) -> /H5_7
- H1 pad 89: unconnected-(H2-Pad89) -> /H5_6
- H1 pad 90: unconnected-(H2-Pad90) -> /H2_18
- H1 pad 91: unconnected-(H2-Pad91) -> /H2_17
- H1 pad 92: unconnected-(H2-Pad92) -> /H5_18
- H1 pad 93: unconnected-(H2-Pad93) -> /H5_19
- H1 pad 94: unconnected-(H2-Pad94) -> /PROG_PIN
- H2 pad 1: unconnected-(H1-Pad1) -> GND
- H2 pad 10: unconnected-(H1-Pad10) (its old number) -> /VCC3
- H2 pad 11: unconnected-(H1-Pad11) -> /VCC2_OUT
- H2 pad 12: unconnected-(H1-Pad12) -> /H2_12
- H2 pad 13: unconnected-(H1-Pad13) -> /H2_13
- H2 pad 14: unconnected-(H1-Pad14) -> /H2_14
- H2 pad 15: unconnected-(H1-Pad15) (its old number) -> /H2_15
- H2 pad 16: unconnected-(H1-Pad16) (its old number) -> /H2_16
- H2 pad 17: unconnected-(H1-Pad17) -> /H2_17
- H2 pad 18: unconnected-(H1-Pad18) (its old number) -> /H2_18
- H2 pad 19: unconnected-(H1-Pad19) (its old number) -> /H2_19
- H2 pad 20: unconnected-(H1-Pad20) (its old number) -> GND
- H2 pad 3: unconnected-(H1-Pad3) (its old number) -> Net-(H2-Pad3)
- H2 pad 4: unconnected-(H1-Pad4) -> Net-(H2-Pad4)
- H2 pad 5: unconnected-(H1-Pad5) -> Net-(H2-Pad5)
- H2 pad 6: unconnected-(H1-Pad6) -> /H2_6
- H2 pad 7: unconnected-(H1-Pad7) -> /H2_7
- H2 pad 8: unconnected-(H1-Pad8) (its old number) -> /H2_8
- H2 pad 9: unconnected-(H1-Pad9) (its old number) -> /H2_9
- H3 pad 1: unconnected-(H3-Pad1) -> GND
- H3 pad 10: unconnected-(H3-Pad10) -> /VCC3
- H3 pad 11: unconnected-(H3-Pad11) -> /VCC2_OUT
- H3 pad 12: unconnected-(H3-Pad12) -> /H3_12
- H3 pad 13: unconnected-(H3-Pad13) -> /H3_13
- H3 pad 14: unconnected-(H3-Pad14) -> /H3_14
- H3 pad 15: unconnected-(H3-Pad15) -> /H3_15
- H3 pad 16: unconnected-(H3-Pad16) -> /H3_16
- H3 pad 17: unconnected-(H3-Pad17) -> /H3_17
- H3 pad 18: unconnected-(H3-Pad18) -> /H3_18
- H3 pad 19: unconnected-(H3-Pad19) -> /H3_19
- H3 pad 2: unconnected-(H3-Pad2) -> Net-(H3-Pad2)
- H3 pad 20: unconnected-(H3-Pad20) -> GND
- H3 pad 3: unconnected-(H3-Pad3) -> Net-(H3-Pad3)
- H3 pad 4: unconnected-(H3-Pad4) -> Net-(H3-Pad4)
- H3 pad 5: unconnected-(H3-Pad5) -> Net-(H3-Pad5)
- H3 pad 6: unconnected-(H3-Pad6) -> /H3_6
- H3 pad 7: unconnected-(H3-Pad7) -> /H3_7
- H3 pad 8: unconnected-(H3-Pad8) -> /H3_8
- H3 pad 9: unconnected-(H3-Pad9) -> /H3_9
- H4 pad 1: unconnected-(H4-Pad1) -> GND
- H4 pad 10: unconnected-(H4-Pad10) -> /VCC3
- H4 pad 11: unconnected-(H4-Pad11) -> /VCC2_OUT
- H4 pad 12: unconnected-(H4-Pad12) -> /H3_12
- H4 pad 13: unconnected-(H4-Pad13) -> /H3_13
- H4 pad 14: unconnected-(H4-Pad14) -> /H3_14
- H4 pad 15: unconnected-(H4-Pad15) -> /H4_15
- H4 pad 16: unconnected-(H4-Pad16) -> /H4_16
- H4 pad 17: unconnected-(H4-Pad17) -> /H4_17
- H4 pad 18: unconnected-(H4-Pad18) -> /H4_18
- H4 pad 19: unconnected-(H4-Pad19) -> /H4_19
- H4 pad 2: unconnected-(H4-Pad2) -> Net-(H4-Pad2)
- H4 pad 20: unconnected-(H4-Pad20) -> GND
- H4 pad 3: unconnected-(H4-Pad3) -> Net-(H4-Pad3)
- H4 pad 4: unconnected-(H4-Pad4) -> Net-(H4-Pad4)
- H4 pad 5: unconnected-(H4-Pad5) -> Net-(H4-Pad5)
- H4 pad 6: unconnected-(H4-Pad6) -> /H4_6
- H4 pad 7: unconnected-(H4-Pad7) -> /H4_7
- H4 pad 8: unconnected-(H4-Pad8) -> /H3_8
- H4 pad 9: unconnected-(H4-Pad9) -> /H3_9
- H5 pad 1: unconnected-(H5-Pad1) -> GND
- H5 pad 10: unconnected-(H5-Pad10) -> /VCC3
- H5 pad 11: unconnected-(H5-Pad11) -> /VCC2_OUT
- H5 pad 12: unconnected-(H5-Pad12) -> /H2_12
- H5 pad 13: unconnected-(H5-Pad13) -> /H2_13
- H5 pad 14: unconnected-(H5-Pad14) -> /H2_14
- H5 pad 15: unconnected-(H5-Pad15) -> /H5_15
- H5 pad 16: unconnected-(H5-Pad16) -> /H5_16
- H5 pad 17: unconnected-(H5-Pad17) -> /H5_17
- H5 pad 18: unconnected-(H5-Pad18) -> /H5_18
- H5 pad 19: unconnected-(H5-Pad19) -> /H5_19
- H5 pad 2: unconnected-(H5-Pad2) -> Net-(H5-Pad2)
- H5 pad 20: unconnected-(H5-Pad20) -> GND
- H5 pad 3: unconnected-(H5-Pad3) -> Net-(H5-Pad3)
- H5 pad 4: unconnected-(H5-Pad4) -> Net-(H5-Pad4)
- H5 pad 5: unconnected-(H5-Pad5) -> Net-(H5-Pad5)
- H5 pad 6: unconnected-(H5-Pad6) -> /H5_6
- H5 pad 7: unconnected-(H5-Pad7) -> /H5_7
- H5 pad 8: unconnected-(H5-Pad8) -> /H2_8
- H5 pad 9: unconnected-(H5-Pad9) -> /H2_9
- IC7 pad 1: unconnected-(IC7-PB9-BOOT0-Pad1) -> /PWR_MCU_BOOTLOADER
- IC7 pad 17: unconnected-(IC7-PA9-Pad17) -> /PWR_MCU_I2C_SCL
- IC7 pad 18: unconnected-(IC7-PA10-Pad18) -> /PWR_MCU_I2C_SDA
- J1 pad 3: unconnected-(J1-Pad3) -> Net-(H4-Pad2)
- J1 pad 4: unconnected-(J1-Pad4) -> Net-(H4-Pad3)
- J1 pad 5: unconnected-(J1-Pad5) -> Net-(H4-Pad4)
- J1 pad 6: unconnected-(J1-Pad6) -> Net-(H4-Pad5)
- J2 pad 5: unconnected-(J2-Pad5) -> Net-(H5-Pad4)
- J2 pad 6: unconnected-(J2-Pad6) -> Net-(H5-Pad5)
- J3 pad 5: unconnected-(J3-Pad5) -> Net-(H5-Pad2)
- J3 pad 6: unconnected-(J3-Pad6) -> Net-(H5-Pad3)
- J4 pad 3: unconnected-(J4-Pad3) -> Net-(H3-Pad2)
- J4 pad 4: unconnected-(J4-Pad4) -> Net-(H3-Pad3)
- J4 pad 5: unconnected-(J4-Pad5) -> Net-(H3-Pad4)
- J4 pad 6: unconnected-(J4-Pad6) -> Net-(H3-Pad5)
- J6 pad 3: unconnected-(J6-Pad3) -> /PROG_PIN
- J6 pad 4: unconnected-(J6-Pad4) -> Net-(H2-Pad3)
- J6 pad 5: unconnected-(J6-Pad5) -> Net-(H2-Pad4)
- J6 pad 6: unconnected-(J6-Pad6) -> Net-(H2-Pad5)
Routing:
- net GND: track 344.0 -> 529.2 mm, vias 60 -> 84
- net /VCC2_OUT: track 0.00 -> 173.4 mm, vias 0 -> 6
- net /VCC3: track 45.5 -> 181.9 mm, vias 30 -> 37
- net /PWR_MCU_I2C_SDA: track 0.00 -> 90.5 mm, vias 0 -> 4
- net /PWR_MCU_I2C_SCL: track 0.00 -> 90.0 mm, vias 0 -> 4
- net /H3_9: track 0.00 -> 70.9 mm, vias 0 -> 3
- net /H3_8: track 0.00 -> 70.3 mm, vias 0 -> 3
- net /H3_14: track 0.00 -> 64.2 mm, vias 0 -> 3
- net /H3_13: track 0.00 -> 62.6 mm, vias 0 -> 3
- net /H3_12: track 0.00 -> 60.5 mm, vias 0 -> 3
- net /H3_15: track 0.00 -> 59.5 mm, vias 0 -> 3
- net /PROG_PIN: track 0.00 -> 53.6 mm, vias 0 -> 1
- net /H3_19: track 0.00 -> 53.3 mm, vias 0 -> 3
- net Net-(H4-Pad5): track 0.00 -> 53.3 mm, vias 0 -> 1
- net /H3_18: track 0.00 -> 52.9 mm, vias 0 -> 3
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Other:
- board text added: "+"
- board text added: "1 2 3 4"
- board text added: "G"
- board text added: "PRG."
- board text added: "PWR_IN"
- board text added: "έξυπνο καλώδιο 2 (C.S.C.S.)"
- board text added: "α1"

Commit message: MB V1 finished again
Parts:
- added R53: ERJ-2RKF1002X, SamacSys_Parts:ERJ2RKD1004X, F.Cu at (116.9, 143.6)
- added R54: ERJ-2RKF1002X, SamacSys_Parts:ERJ2RKD1004X, F.Cu at (123.4, 142.0)
- added R55: ERJ-2RKF1002X, SamacSys_Parts:ERJ2RKD1004X, F.Cu at (131.7, 142.0)
- added R56: ERJ-2RKF1002X, SamacSys_Parts:ERJ2RKD1004X, F.Cu at (140.1, 142.0)
- added R57: ERJ-2RKF1002X, SamacSys_Parts:ERJ2RKD1004X, F.Cu at (149.3, 142.0)
Routing:
- net GND: track 529.2 -> 541.8 mm, vias 84 -> 88
- net /S1_SW_EN: track 45.1 -> 48.3 mm
- net /S2_SW_EN: track 38.2 -> 40.4 mm
- net /S4_SW_EN: track 24.0 -> 26.2 mm
- net /S3_SW_EN: track 30.9 -> 33.1 mm
- net /S5_SW_EN: track 14.4 -> 16.1 mm
- net /S1_SW_IMON: track 46.5 -> 48.1 mm
- net /H3_17: track 48.6 -> 49.8 mm
- net /H3_16: track 49.5 -> 50.7 mm
- net /PWR_MCU_I2C_SCL: track 90.0 -> 90.6 mm
- net /PWR_MCU_I2C_SDA: track 90.5 -> 91.0 mm
