File: motherboard/V1/MB_V1.kicad_sch (KiCad schematic)
At the start: 85 parts, among them IC1 TPS27S100BRRKR, IC2 TPS27S100BRRKR, IC3 TPS27S100BRRKR, IC4 TPS27S100BRRKR, IC5 TPS27S100BRRKR, IC7 STM32L010F4P6TR, J1 640456-6, J2 640456-6, J3 640456-6, J4 640456-6, J5 640454-2, J6 640456-6, Q1 SQS141ELNW-T1_GE3

Commit message: MB V1 finished
Parts:
- added C11: C0603C104K5RAC3121, CAPC1608X95N, symbol SamacSys_Parts:C0603C104K5RAC3121
- added Q1: IRLML6244TRPBF, SOT95P237X112-3N, symbol SamacSys_Parts:IRLML6244TRPBF
- added R4: ERJ2RKF1003X, ERJ2RKD1004X, symbol SamacSys_Parts:ERJ2RKF1003X
- added R48: WSL080500000ZEA9, RESC2013X84N, symbol SamacSys_Parts:WSL080500000ZEA9
- added R50, R51, R52: ERJ-2RKF1002X, ERJ2RKD1004X, symbol SamacSys_Parts:ERJ-2RKF1002X
- renumbered H2 to H1, H1 to H2
Connections:
- net GND: now also H1.100, H1.25, H1.50, H1.51, H1.75, H1.76, H2.1, H2.20, H3.1, H3.20, H4.1, H4.20, H5.1, H5.20, Q1.2 (S), R4.1, R50.1
- net VCC2: now also R48.2
- net VCC3: now also H1.1, H1.2, H2.10, H3.10, H4.10, H5.10
- net at J3.5: now also H5.2
- net at J3.6: now also H5.3
- net VCC2_OUT: now reaches H2.11
- net VCC2_OUT: now also H1.26, H3.11, H4.11, H5.11, R48.1
- net H2_12: now reaches H2.12
- net H2_12: now also H1.84, H5.12
- net H2_13: now reaches H2.13
- net H2_13: now also H1.83, H5.13
- net H2_14: now reaches H2.14
- net H2_14: now also H1.82, H5.14
- net H2_15: now reaches H2.15
- net H2_15: now also H1.79
- net H2_16: now reaches H2.16
- net H2_16: now also H1.78
- net H2_17: now reaches H2.17
- net H2_17: now also H1.91
- net H2_18: now reaches H2.18
- net H2_18: now also H1.90
- net H2_19: now reaches H2.19
- net H2_19: now also H1.85
- net at H2.3: now also J6.4
- net at H2.4: now also J6.5
- net at H2.5: now also J6.6
- net H2_6: now reaches H2.6
- net H2_6: now also H1.87
- net H2_7: now reaches H2.7
- net H2_7: now also H1.86
- net H2_8: now reaches H2.8
- net H2_8: now also H1.55, H5.8
- net H2_9: now reaches H2.9
- net H2_9: now also H1.54, H5.9
- net PWR_MCU_BOOTLOADER: now reaches IC7.1 (PB9-BOOT0)
- net PWR_MCU_BOOTLOADER: now also H1.7, C11.2, R50.2
- net PWR_MCU_I2C_SCL: now reaches IC7.17 (PA9)
- net PWR_MCU_I2C_SCL: now also H1.65, R51.1
- net PWR_MCU_I2C_SDA: now reaches IC7.18 (PA10)
- net PWR_MCU_I2C_SDA: now also H1.64, R52.1
- net at IC7.4 (NRST), R32.1: now also Q1.3 (D)
- net at J1.3: now also H4.2
- net at J1.4: now also H4.3
- net at J1.5: now also H4.4
- net at J1.6: now also H4.5
- net H3_12: now reaches H3.12
- net H3_12: now also H1.32, H4.12
- net H3_13: now reaches H3.13
- net H3_13: now also H1.31, H4.13
- net H3_14: now reaches H3.14
- net H3_14: now also H1.30, H4.14
- net H3_15: now reaches H3.15
- net H3_15: now also H1.40
- net H3_16: now reaches H3.16
- net H3_16: now also H1.62
- net H3_17: now reaches H3.17
- net H3_17: now also H1.61
- net H3_18: now reaches H3.18
- net H3_18: now also H1.12
- net H3_19: now reaches H3.19
- net H3_19: now also H1.11
- net at H3.2: now also J4.3
- net at H3.3: now also J4.4
- net at H3.4: now also J4.5
- net at H3.5: now also J4.6
- net H3_6: now reaches H3.6
- net H3_6: now also H1.81
- net H3_7: now reaches H3.7
- net H3_7: now also H1.80
- net H3_8: now reaches H3.8
- net H3_8: now also H1.14, H4.8
- net H3_9: now reaches H3.9
- net H3_9: now also H1.13, H4.9
- net at J2.5: now also H5.4
- net at J2.6: now also H5.5
- net H5_15: now reaches H5.15
- net H5_15: now also H1.68
- net H5_16: now reaches H5.16
- net H5_16: now also H1.67
- net H5_17: now reaches H5.17
- net H5_17: now also H1.66
- net H5_18: now reaches H5.18
- net H5_18: now also H1.92
- net H5_19: now reaches H5.19
- net H5_19: now also H1.93
- net H5_6: now reaches H5.6
- net H5_6: now also H1.89
- net H5_7: now reaches H5.7
- net H5_7: now also H1.88
- net H4_15: now reaches H4.15
- net H4_15: now also H1.6
- net H4_16: now reaches H4.16
- net H4_16: now also H1.5
- net H4_17: now reaches H4.17
- net H4_17: now also H1.4
- net H4_18: now reaches H4.18
- net H4_18: now also H1.37
- net H4_19: now reaches H4.19
- net H4_19: now also H1.36
- net H4_6: now reaches H4.6
- net H4_6: now also H1.39
- net H4_7: now reaches H4.7
- net H4_7: now also H1.38
- net PROG_PIN: now reaches J6.3
- net PROG_PIN: now also H1.94
- net PWR_I2C_PULLUP: now reaches H1.17
- net PWR_I2C_PULLUP: now also R51.2, R52.2
- new net: C11.1, Q1.1 (G), R4.2
Other:
- note added: "INTERFACE MODULES"
- note added: "MCU MODULE"
- note added: "PORT POWER SWITCHES"
- note added: "POWER CONTROLLER"
- note added: "SENSORS CONNECTORS"
- moved on the sheet: C1, C10, C11, C12, C2, C3, C4, C5, C6, C7, C8, C9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

Commit message: MB V1 finished again
Parts:
- added R53, R54, R55, R56, R57: ERJ-2RKF1002X, ERJ2RKD1004X, symbol SamacSys_Parts:ERJ-2RKF1002X
Connections:
- net GND: now also R53.1, R54.1, R55.1, R56.1, R57.1
- net S1_SW_EN: now also R53.2
- net S2_SW_EN: now also R54.2
- net S3_SW_EN: now also R55.2
- net S4_SW_EN: now also R56.2
- net S5_SW_EN: now also R57.2
