File: modules/RS232-2/α1/RS232-2_α1.kicad_pcb (KiCad board)
At the start: 2 copper layers, 20 x 20 mm, 14 parts, among them IC1 MAX3221EAE+, IC2 MAX3221EAE+

Commit message: IMU added
Connections:
- net /VCC2 renamed /VCC3
Changed lines of the file:
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@@
       (usegerberattributes true)
       (usegerberadvancedattributes true)
-      (creategerberjobfile true)
+      (creategerberjobfile false)
       (dashed_line_dash_ratio 12.000000)
       (dashed_line_gap_ratio 3.000000)
@@
   (net 9 "/UART_A_TTL_TX")
   (net 10 "/UART_A_TTL_RX")
-  (net 11 "/VCC2")
+  (net 11 "/VCC3")
   (net 12 "/UART_B_TTL_TX")
   (net 13 "/UART_B_TTL_RX")
@@
     (property "Mouser Part Number" "80-C603C104K5RAC3121")
     (property "Mouser Price/Stock" "https://www.mouser.co.uk/ProductDetail/KEMET/C0603C104K5RAC3121?qs=oBCMsStVSxe1EkGyoyETtg%3D%3D")
-    (property "Sheetfile" "RS232_α1.kicad_sch")
+    (property "Sheetfile" "RS232-2_α1.kicad_sch")
     (property "Sheetname" "")
     (property "ki_description" "Multilayer Ceramic Capacitors MLCC - SMD/SMT 50V .1uF X7R 0603 10% AEC-Q200")
@@
     (property "Mouser Part Number" "80-C603C104K5RAC3121")
     (property "Mouser Price/Stock" "https://www.mouser.co.uk/ProductDetail/KEMET/C0603C104K5RAC3121?qs=oBCMsStVSxe1EkGyoyETtg%3D%3D")
-    (property "Sheetfile" "RS232_α1.kicad_sch")
+    (property "Sheetfile" "RS232-2_α1.kicad_sch")
     (property "Sheetname" "")
     (property "ki_description" "Multilayer Ceramic Capacitors MLCC - SMD/SMT 50V .1uF X7R 0603 10% AEC-Q200")
@@
     (property "Mouser Part Number" "80-C603C104K5RAC3121")
     (property "Mouser Price/Stock" "https://www.mouser.co.uk/ProductDetail/KEMET/C0603C104K5RAC3121?qs=oBCMsStVSxe1EkGyoyETtg%3D%3D")
-    (property "Sheetfile" "RS232_α1.kicad_sch")
+    (property "Sheetfile" "RS232-2_α1.kicad_sch")
     (property "Sheetname" "")
     (property "ki_description" "Multilayer Ceramic Capacitors MLCC - SMD/SMT 50V .1uF X7R 0603 10% AEC-Q200")
@@
     (property "Mouser Part Number" "80-C603C104K5RAC3121")
     (property "Mouser Price/Stock" "https://www.mouser.co.uk/ProductDetail/KEMET/C0603C104K5RAC3121?qs=oBCMsStVSxe1EkGyoyETtg%3D%3D")
-    (property "Sheetfile" "RS232_α1.kicad_sch")
+    (property "Sheetfile" "RS232-2_α1.kicad_sch")
     (property "Sheetname" "")
     (property "ki_description" "Multilayer Ceramic Capacitors MLCC - SMD/SMT 50V .1uF X7R 0603 10% AEC-Q200")
@@
       (net 8 "GND") (pintype "passive") (thermal_bridge_angle 45))
     (pad "2" smd rect (at 0.7 0 90) (size 0.78 0.98) (layers "F.Cu" "F.Paste" "F.Mask")
-      (net 11 "/VCC2") (pintype "passive") (thermal_bridge_angle 45))
+      (net 11 "/VCC3") (pintype "passive") (thermal_bridge_angle 45))
   )
   (footprint "SamacSys_Parts:CAPC1608X95N" (layer "F.Cu")
@@
     (property "Mouser Part Number" "80-C603C104K5RAC3121")
     (property "Mouser Price/Stock" "https://www.mouser.co.uk/ProductDetail/KEMET/C0603C104K5RAC3121?qs=oBCMsStVSxe1EkGyoyETtg%3D%3D")
-    (property "Sheetfile" "RS232_α1.kicad_sch")
+    (property "Sheetfile" "RS232-2_α1.kicad_sch")
     (property "Sheetname" "")
     (property "ki_description" "Multilayer Ceramic Capacitors MLCC - SMD/SMT 50V .1uF X7R 0603 10% AEC-Q200")
@@
     (property "Mouser Part Number" "80-C603C104K5RAC3121")
     (property "Mouser Price/Stock" "https://www.mouser.co.uk/ProductDetail/KEMET/C0603C104K5RAC3121?qs=oBCMsStVSxe1EkGyoyETtg%3D%3D")
-    (property "Sheetfile" "RS232_α1.kicad_sch")
+    (property "Sheetfile" "RS232-2_α1.kicad_sch")
     (property "Sheetname" "")
     (property "ki_description" "Multilayer Ceramic Capacitors MLCC - SMD/SMT 50V .1uF X7R 0603 10% AEC-Q200")
@@
     (property "Mouser Part Number" "80-C603C104K5RAC3121")
     (property "Mouser Price/Stock" "https://www.mouser.co.uk/ProductDetail/KEMET/C0603C104K5RAC3121?qs=oBCMsStVSxe1EkGyoyETtg%3D%3D")
-    (property "Sheetfile" "RS232_α1.kicad_sch")
+    (property "Sheetfile" "RS232-2_α1.kicad_sch")
     (property "Sheetname" "")
     (property "ki_description" "Multilayer Ceramic Capacitors MLCC - SMD/SMT 50V .1uF X7R 0603 10% AEC-Q200")
@@
       (net 8 "GND") (pintype "passive") (thermal_bridge_angle 45))
     (pad "2" smd rect (at 0.7 0 90) (size 0.78 0.98) (layers "F.Cu" "F.Paste" "F.Mask")
-      (net 11 "/VCC2") (pintype "passive") (thermal_bridge_angle 45))
+      (net 11 "/VCC3") (pintype "passive") (thermal_bridge_angle 45))
   )
   (footprint "SamacSys_Parts:SOP65P778X199-16N" (layer "F.Cu")
@@
     (property "Mouser Part Number" "700-MAX3221EAE")
     (property "Mouser Price/Stock" "https://www.mouser.co.uk/ProductDetail/Analog-Devices-Maxim-Integrated/MAX3221EAE%2b?qs=1THa7WoU59EPTKLIY53fFA%3D%3D")
-    (property "Sheetfile" "RS232_α1.kicad_sch")
+    (property "Sheetfile" "RS232-2_α1.kicad_sch")
     (property "Sheetname" "")
     (property "ki_description" "MAX3221EAE+, Line Transceiver 1 1 1 235 kbit/s, 3  5.5 V, 16-Pin SSOP")
@@
       (net 8 "GND") (pinfunction "GND") (pintype "passive") (thermal_bridge_angle 45))
     (pad "15" smd rect (at 3.498 -1.625 90) (size 0.45 1.705) (layers "F.Cu" "F.Paste" "F.Mask")
-      (net 11 "/VCC2") (pinfunction "VCC") (pintype "passive") (thermal_bridge_angle 45))
+      (net 11 "/VCC3") (pinfunction "VCC") (pintype "passive") (thermal_bridge_angle 45))
     (pad "16" smd rect (at 3.498 -2.275 90) (size 0.45 1.705) (layers "F.Cu" "F.Paste" "F.Mask")
-      (net 11 "/VCC2") (pinfunction "~{FORCEOFF}") (pintype "passive") (thermal_bridge_angle 45))
+      (net 11 "/VCC3") (pinfunction "~{FORCEOFF}") (pintype "passive") (thermal_bridge_angle 45))
   )
   (footprint "SamacSys_Parts:CAPC1608X95N" (layer "F.Cu")
@@
     (property "Mouser Part Number" "80-C603C104K5RAC3121")
     (property "Mouser Price/Stock" "https://www.mouser.co.uk/ProductDetail/KEMET/C0603C104K5RAC3121?qs=oBCMsStVSxe1EkGyoyETtg%3D%3D")
-    (property "Sheetfile" "RS232_α1.kicad_sch")
+    (property "Sheetfile" "RS232-2_α1.kicad_sch")
     (property "Sheetname" "")
     (property "ki_description" "Multilayer Ceramic Capacitors MLCC - SMD/SMT 50V .1uF X7R 0603 10% AEC-Q200")
@@
     (property "Mouser Part Number" "80-C603C104K5RAC3121")
     (property "Mouser Price/Stock" "https://www.mouser.co.uk/ProductDetail/KEMET/C0603C104K5RAC3121?qs=oBCMsStVSxe1EkGyoyETtg%3D%3D")
-    (property "Sheetfile" "RS232_α1.kicad_sch")
+    (property "Sheetfile" "RS232-2_α1.kicad_sch")
     (property "Sheetname" "")
     (property "ki_description" "Multilayer Ceramic Capacitors MLCC - SMD/SMT 50V .1uF X7R 0603 10% AEC-Q200")
@@
     (property "Mouser Part Number" "80-C603C104K5RAC3121")
     (property "Mouser Price/Stock" "https://www.mouser.co.uk/ProductDetail/KEMET/C0603C104K5RAC3121?qs=oBCMsStVSxe1EkGyoyETtg%3D%3D")
-    (property "Sheetfile" "RS232_α1.kicad_sch")
+    (property "Sheetfile" "RS232-2_α1.kicad_sch")
     (property "Sheetname" "")
     (property "ki_description" "Multilayer Ceramic Capacitors MLCC - SMD/SMT 50V .1uF X7R 0603 10% AEC-Q200")
@@
     (property "Mouser Part Number" "700-MAX3221EAE")
     (property "Mouser Price/Stock" "https://www.mouser.co.uk/ProductDetail/Analog-Devices-Maxim-Integrated/MAX3221EAE%2b?qs=1THa7WoU59EPTKLIY53fFA%3D%3D")
-    (property "Sheetfile" "RS232_α1.kicad_sch")
+    (property "Sheetfile" "RS232-2_α1.kicad_sch")
     (property "Sheetname" "")
     (property "ki_description" "MAX3221EAE+, Line Transceiver 1 1 1 235 kbit/s, 3  5.5 V, 16-Pin SSOP")
@@
       (net 8 "GND") (pinfunction "GND") (pintype "passive") (thermal_bridge_angle 45))
     (pad "15" smd rect (at 3.498 -1.625 90) (size 0.45 1.705) (layers "F.Cu" "F.Paste" "F.Mask")
-      (net 11 "/VCC2") (pinfunction "VCC") (pintype "passive") (thermal_bridge_angle 45))
+      (net 11 "/VCC3") (pinfunction "VCC") (pintype "passive") (thermal_bridge_angle 45))
     (pad "16" smd rect (at 3.498 -2.275 90) (size 0.45 1.705) (layers "F.Cu" "F.Paste" "F.Mask")
-      (net 11 "/VCC2") (pinfunction "~{FORCEOFF}") (pintype "passive") (thermal_bridge_angle 45))
+      (net 11 "/VCC3") (pinfunction "~{FORCEOFF}") (pintype "passive") (thermal_bridge_angle 45))
   )
   (footprint "USIB2:IF_2020_20_MODULE_FX6" (layer "B.Cu")
     (at 114.94 88.78 -90)
     (property "Connector" "FX620P08SV")
-    (property "Sheetfile" "RS232_α1.kicad_sch")
+    (property "Sheetfile" "RS232-2_α1.kicad_sch")
     (property "Sheetname" "")
     (attr smd)
@@
       (net 2 "unconnected-(H1-Pad9)") (pintype "passive") (thermal_bridge_angle 45))
     (pad "10" smd rect (at -3.6 -2.6 270) (size 0.5 2) (layers "B.Cu" "B.Paste" "B.Mask")
-      (net 11 "/VCC2") (pintype "passive") (thermal_bridge_angle 45))
+      (net 11 "/VCC3") (pintype "passive") (thermal_bridge_angle 45))
     (pad "11" smd rect (at -3.6 -7.3 270) (size 0.5 2) (layers "B.Cu" "B.Paste" "B.Mask")
       (net 3 "unconnected-(H1-Pad11)") (pintype "passive") (thermal_bridge_angle 45))
