File: modules/RS232-2/α1/RS232-2_α1.kicad_sch (KiCad schematic)
At the start: 13 parts, among them IC1 MAX3221EAE+, IC2 MAX3221EAE+

Commit message: IMU added
Connections:
- net VCC2 renamed VCC3
Changed lines of the file:
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@@
     (effects (font (size 1.27 1.27)) (justify left bottom))
   )
-  (label "VCC2" (at 143.002 137.414 0) (fields_autoplaced)
+  (label "VCC3" (at 143.002 137.414 0) (fields_autoplaced)
     (effects (font (size 1.27 1.27)) (justify left bottom))
   )
@@
     (effects (font (size 1.27 1.27)) (justify left bottom))
   )
-  (label "VCC2" (at 255.143 61.341 0) (fields_autoplaced)
+  (label "VCC3" (at 255.143 61.341 0) (fields_autoplaced)
     (effects (font (size 1.27 1.27)) (justify left bottom))
   )
-  (label "VCC2" (at 49.7586 48.641 0) (fields_autoplaced)
+  (label "VCC3" (at 49.7586 48.641 0) (fields_autoplaced)
     (effects (font (size 1.27 1.27)) (justify left bottom))
   )
@@
     (pin "2")
     (instances
-      (project "RS232_α1"
+      (project "RS232-2_α1"
         (path "/a97216d2-ea19-4316-99be-5ed65c12da81"
           (reference "C1") (unit 1)
@@
     (pin "2")
     (instances
-      (project "RS232_α1"
+      (project "RS232-2_α1"
         (path "/a97216d2-ea19-4316-99be-5ed65c12da81"
           (reference "C8") (unit 1)
@@
     (pin "1")
     (instances
-      (project "RS232_α1"
+      (project "RS232-2_α1"
         (path "/a97216d2-ea19-4316-99be-5ed65c12da81"
           (reference "#PWR05") (unit 1)
@@
     (pin "2")
     (instances
-      (project "RS232_α1"
+      (project "RS232-2_α1"
         (path "/a97216d2-ea19-4316-99be-5ed65c12da81"
           (reference "C3") (unit 1)
@@
     (pin "2")
     (instances
-      (project "RS232_α1"
+      (project "RS232-2_α1"
         (path "/a97216d2-ea19-4316-99be-5ed65c12da81"
           (reference "C10") (unit 1)
@@
     (pin "9")
     (instances
-      (project "RS232_α1"
+      (project "RS232-2_α1"
         (path "/a97216d2-ea19-4316-99be-5ed65c12da81"
           (reference "IC2") (unit 1)
@@
     (pin "1")
     (instances
-      (project "RS232_α1"
+      (project "RS232-2_α1"
         (path "/a97216d2-ea19-4316-99be-5ed65c12da81"
           (reference "#PWR03") (unit 1)
@@
     (pin "2")
     (instances
-      (project "RS232_α1"
+      (project "RS232-2_α1"
         (path "/a97216d2-ea19-4316-99be-5ed65c12da81"
           (reference "C4") (unit 1)
@@
     (pin "2")
     (instances
-      (project "RS232_α1"
+      (project "RS232-2_α1"
         (path "/a97216d2-ea19-4316-99be-5ed65c12da81"
           (reference "C7") (unit 1)
@@
     (pin "2")
     (instances
-      (project "RS232_α1"
+      (project "RS232-2_α1"
         (path "/a97216d2-ea19-4316-99be-5ed65c12da81"
           (reference "C6") (unit 1)
@@
     (pin "2")
     (instances
-      (project "RS232_α1"
+      (project "RS232-2_α1"
         (path "/a97216d2-ea19-4316-99be-5ed65c12da81"
           (reference "C2") (unit 1)
@@
     (pin "1")
     (instances
-      (project "RS232_α1"
+      (project "RS232-2_α1"
         (path "/a97216d2-ea19-4316-99be-5ed65c12da81"
           (reference "#PWR09") (unit 1)
@@
     (pin "1")
     (instances
-      (project "RS232_α1"
+      (project "RS232-2_α1"
         (path "/a97216d2-ea19-4316-99be-5ed65c12da81"
           (reference "#PWR011") (unit 1)
@@
     (pin "9")
     (instances
-      (project "RS232_α1"
+      (project "RS232-2_α1"
         (path "/a97216d2-ea19-4316-99be-5ed65c12da81"
           (reference "H1") (unit 1)
@@
     (pin "9")
     (instances
-      (project "RS232_α1"
+      (project "RS232-2_α1"
         (path "/a97216d2-ea19-4316-99be-5ed65c12da81"
           (reference "IC1") (unit 1)
@@
     (pin "1")
     (instances
-      (project "RS232_α1"
+      (project "RS232-2_α1"
         (path "/a97216d2-ea19-4316-99be-5ed65c12da81"
           (reference "#PWR06") (unit 1)
@@
     (pin "1")
     (instances
-      (project "RS232_α1"
+      (project "RS232-2_α1"
         (path "/a97216d2-ea19-4316-99be-5ed65c12da81"
           (reference "#PWR010") (unit 1)
@@
     (pin "1")
     (instances
-      (project "RS232_α1"
+      (project "RS232-2_α1"
         (path "/a97216d2-ea19-4316-99be-5ed65c12da81"
           (reference "#PWR04") (unit 1)
@@
     (pin "1")
     (instances
-      (project "RS232_α1"
+      (project "RS232-2_α1"
         (path "/a97216d2-ea19-4316-99be-5ed65c12da81"
           (reference "#PWR07") (unit 1)
@@
     (pin "1")
     (instances
-      (project "RS232_α1"
+      (project "RS232-2_α1"
         (path "/a97216d2-ea19-4316-99be-5ed65c12da81"
           (reference "#PWR08") (unit 1)
@@
     (pin "1")
     (instances
-      (project "RS232_α1"
+      (project "RS232-2_α1"
         (path "/a97216d2-ea19-4316-99be-5ed65c12da81"
           (reference "#PWR01") (unit 1)
@@
     (pin "2")
     (instances
-      (project "RS232_α1"
+      (project "RS232-2_α1"
         (path "/a97216d2-ea19-4316-99be-5ed65c12da81"
           (reference "C5") (unit 1)
@@
     (pin "2")
     (instances
-      (project "RS232_α1"
+      (project "RS232-2_α1"
         (path "/a97216d2-ea19-4316-99be-5ed65c12da81"
           (reference "C9") (unit 1)
@@
     (pin "1")
     (instances
-      (project "RS232_α1"
+      (project "RS232-2_α1"
         (path "/a97216d2-ea19-4316-99be-5ed65c12da81"
           (reference "#PWR02") (unit 1)
